Commit message: Add RVIZ Code, Remove Function and Change Variables add RVIZ code:   about 11th robot remove function:   remove initParameterPath function and related variable change variables:   STANDPATH => tool->standPath   parameter_path => tool->parameterPath

File: urdf/kidsize_model/11th/robots/11th.xacro (robot description, xacro)
@@ -351,5 +351,5 @@
       link="left_upper_arm_link" />
     <axis
-      xyz="1 0 0" />
+      xyz="-1 0 0" />
     <limit
       lower="${-pi*0.9}"
@@ -595,5 +595,5 @@
       link="right_upper_arm_link" />
     <axis
-      xyz="1 0 0" />
+      xyz="-1 0 0" />
     <limit
       lower="${-pi*0.9}"
@@ -1532,4 +1532,37 @@
     </inertial>
   </link>
+  <joint
+    name="camera_joint"
+    type="fixed">
+    <origin
+      xyz="0.00225 -4.4516E-05 0.0385"
+      rpy="0 0 0" />
+    <parent
+      link="head_link" />
+    <child
+      link="camera_link" />
+    <axis
+      xyz="0 0 0" />
+  </joint>
+  <!-- Camera -->
+  <link name="camera_link">
+    <collision>
+      <origin xyz="-0.006 0 0" rpy="0 1.5708 0"/>
+      <geometry>
+    <cylinder radius="0.0001" length="0.0005"/>
+      </geometry>
+    </collision>
+    <visual>
+      <origin xyz="-0.006 0 0" rpy="0 1.5708 0"/>
+      <geometry>
+    <cylinder radius="0.0001" length="0.0005"/>
+      </geometry>
+    </visual>
+    <inertial>
+      <mass value="1e-5" />
+      <origin xyz="0 0 0" rpy="0 0 0"/>
+      <inertia ixx="1e-6" ixy="0" ixz="0" iyy="1e-6" iyz="0" izz="1e-6" />
+    </inertial>
+  </link>
       <transmission name="right_hip_yaw_transmission">
 			  <type>transmission_interface/SimpleTransmission</type>
@@ -1746,4 +1779,23 @@
 			</plugin>
 		</gazebo>
+<gazebo reference="imu_link">
+    <gravity>true</gravity>
+    <sensor name="imu_sensor" type="imu">
+      <always_on>true</always_on>
+      <update_rate>100</update_rate>
+      <visualize>true</visualize>
+      <topic>__default_topic__</topic>
+      <plugin filename="libgazebo_ros_imu_sensor.so" name="imu_plugin">
+        <topicName>imu</topicName>
+        <bodyName>imu_link</bodyName>
+        <updateRateHZ>100.0</updateRateHZ>
+        <gaussianNoise>0.0</gaussianNoise>
+        <xyzOffset>0 0 0</xyzOffset>
+        <rpyOffset>0 0 0</rpyOffset>
+        <frameName>imu_link</frameName>
+      </plugin>
+      <pose>0 0 0 0 0 0</pose>
+    </sensor>
+  </gazebo>
 <gazebo reference="camera_link">
 <material>Gazebo/Black</material>
@@ -1814,6 +1866,6 @@
 			<kp>1000000.0</kp>
 			<kd>100.0</kd>
-			<mu1>10000.0</mu1>
-			<mu2>10000.0</mu2>
+			<mu1>100000.0</mu1>
+			<mu2>100000.0</mu2>
 			<fdir1>1 0 0</fdir1>
 			<maxVel>1.0</maxVel>
@@ -1851,6 +1903,6 @@
 			<kp>1000000.0</kp>
 			<kd>100.0</kd>
-			<mu1>10000.0</mu1>
-			<mu2>10000.0</mu2>
+			<mu1>100000.0</mu1>
+			<mu2>100000.0</mu2>
 			<fdir1>1 0 0</fdir1>
 			<maxVel>1.0</maxVel>

File: urdf/kidsize_model/11th/robots/11th_fake_link.xacro (robot description, xacro)
@@ -1282,4 +1282,63 @@
       damping="0.0"
       friction="0.7" />
+  </joint>
+  <link
+    name="right_bottom_foot_fake_link"><inertial>
+      <origin
+        xyz="0.0832407016442707 -0.0275030808874214 -0.0302963318842118"
+        rpy="0 0 0" />
+      <mass
+        value="0.0001" />
+      <inertia
+        ixx="1.04719755119654E-22"
+        ixy="-1.06581097908222E-67"
+        ixz="3.63206357723254E-51"
+        iyy="1.04719755119654E-22"
+        iyz="-3.03551380010738E-55"
+        izz="1.57079632679485E-22" />
+    </inertial>
+    <visual>
+      <origin
+        xyz="0 0 0"
+        rpy="0 0 0" />
+      <geometry>
+        <mesh
+          filename="package://urdf/kidsize_model/robocup_robot/meshes/right_bottom_foot_fake_link.STL" />
+      </geometry>
+      <material
+        name="">
+        <color
+          rgba="0.792156862745098 0.819607843137255 0.933333333333333 1" />
+      </material>
+    </visual>
+    <collision>
+      <origin
+        xyz="0 0 0"
+        rpy="0 0 0" />
+      <geometry>
+        <mesh
+          filename="package://urdf/kidsize_model/robocup_robot/meshes/right_bottom_foot_fake_link.STL" />
+      </geometry>
+    </collision>
+  </link>
+  <joint
+    name="right_bottom_foot_fake_joint"
+    type="fixed">
+    <origin
+      xyz="0.04476 -0.00049 -0.02556"
+      rpy="0 0 0" />
+    <parent
+      link="right_foot_link" />
+    <child
+      link="right_bottom_foot_fake_link" />
+    <axis
+      xyz="1 0 0" />
+    <limit
+      lower="${-pi}"
+      upper="${pi}"
+      effort="10"
+      velocity="0.1" />
+    <dynamics
+      friction="1" />
   </joint>
   <link

Commit message: Fix 11th.xacro error remove imu sensor

File: urdf/kidsize_model/11th/robots/11th.xacro (robot description, xacro)
@@ -1532,5 +1532,5 @@
     </inertial>
   </link>
-  <joint
+  <!-- <joint
     name="camera_joint"
     type="fixed">
@@ -1544,7 +1544,7 @@
     <axis
       xyz="0 0 0" />
-  </joint>
+  </joint> -->
   <!-- Camera -->
-  <link name="camera_link">
+  <!-- <link name="camera_link">
     <collision>
       <origin xyz="-0.006 0 0" rpy="0 1.5708 0"/>
@@ -1564,5 +1564,5 @@
       <inertia ixx="1e-6" ixy="0" ixz="0" iyy="1e-6" iyz="0" izz="1e-6" />
     </inertial>
-  </link>
+  </link> -->
       <transmission name="right_hip_yaw_transmission">
 			  <type>transmission_interface/SimpleTransmission</type>
@@ -1779,5 +1779,5 @@
 			</plugin>
 		</gazebo>
-<gazebo reference="imu_link">
+<!-- <gazebo reference="imu_link">
     <gravity>true</gravity>
     <sensor name="imu_sensor" type="imu">
@@ -1797,5 +1797,5 @@
       <pose>0 0 0 0 0 0</pose>
     </sensor>
-  </gazebo>
+  </gazebo> -->
 <gazebo reference="camera_link">
 <material>Gazebo/Black</material>
