Commit message: new gazebo

File: urdf/kidsize_model/11th/robots/11th.xacro (robot description, xacro)
@@ -2,5 +2,5 @@
 <robot
   name="kidsize" xmlns:xacro="http://www.ros.org/wiki/xacro">
-	<xacro:property name="pi" value="3.14159265359" />
+  <xacro:property name="pi" value="3.14159265359" />
 	<xacro:property name="deg" value="${pi/180}" />
 		<material name="black">
@@ -20,15 +20,15 @@
     <inertial>
       <origin
-        xyz="-0.0153104529258689 0.000169028868324945 -0.00106697942105624"
-        rpy="0 0 0" />
-      <mass
-        value="0.167276714976747" />
-      <inertia
-        ixx="0.000252814781419096"
-        ixy="-1.25057676582085E-06"
-        ixz="-4.84752858921046E-06"
-        iyy="7.39693035453425E-05"
-        iyz="5.2522748791712E-08"
-        izz="0.000281750752840626" />
+        xyz="-0.0088172 -4.3153E-08 -0.0020413"
+        rpy="0 0 0" />
+      <mass
+        value="0.5" />
+      <inertia
+        ixx="0.00037837"
+        ixy="1.6316E-10"
+        ixz="4.0465E-06"
+        iyy="0.00011027"
+        iyz="1.9797E-11"
+        izz="0.00039153" />
     </inertial>
     <visual>
@@ -43,5 +43,5 @@
         name="">
         <color
-          rgba="0.752941176470588 0.752941176470588 0.752941176470588 1" />
+          rgba="0.79216 0.81961 0.93333 1" />
       </material>
     </visual>
@@ -60,15 +60,15 @@
     <inertial>
       <origin
-        xyz="0.00714619272928631 -2.78359236166419E-05 0.108313816832884"
-        rpy="0 0 0" />
-      <mass
-        value="0.264498687306666" />
-      <inertia
-        ixx="0.00102736547091334"
-        ixy="-3.4889421288343E-07"
-        ixz="-3.61057957945358E-05"
-        iyy="0.000786433053168132"
-        iyz="-1.44740860367013E-07"
-        izz="0.000615489834750468" />
+        xyz="0.0077094 2.1697E-05 0.11416"
+        rpy="0 0 0" />
+      <mass
+        value="1.3" />
+      <inertia
+        ixx="0.0010729"
+        ixy="2.0691E-07"
+        ixz="-2.0835E-05"
+        iyy="0.00069595"
+        iyz="4.0117E-07"
+        izz="0.00069847" />
     </inertial>
     <visual>
@@ -83,5 +83,5 @@
         name="">
         <color
-          rgba="0.792156862745098 0.819607843137255 0.933333333333333 1" />
+          rgba="0.79216 0.81961 0.93333 1" />
       </material>
     </visual>
@@ -118,40 +118,40 @@
   </joint>
   <link
-    name="neck_link">
-    <inertial>
-      <origin
-        xyz="-0.00802644264854249 0.000731943028199903 0.0377079510666786"
-        rpy="0 0 0" />
-      <mass
-        value="0.0480257488384161" />
-      <inertia
-        ixx="8.34903166705297E-06"
-        ixy="-1.06975527764787E-07"
-        ixz="-4.74763699335791E-08"
-        iyy="1.34803475325574E-05"
-        iyz="-4.56219872528396E-08"
-        izz="1.41602185792909E-05" />
-    </inertial>
-    <visual>
-      <origin
-        xyz="0 0 0"
-        rpy="0 0 0" />
-      <geometry>
-        <mesh
-          filename="package://urdf/kidsize_model/11th/meshes/neck_link.STL" />
-      </geometry>
-      <material
-        name="">
-        <color
-          rgba="0.792156862745098 0.819607843137255 0.933333333333333 1" />
-      </material>
-    </visual>
-    <collision>
-      <origin
-        xyz="0 0 0"
-        rpy="0 0 0" />
-      <geometry>
-        <mesh
-          filename="package://urdf/kidsize_model/11th/meshes/neck_link.STL" />
+    name="neck_Link">
+    <inertial>
+      <origin
+        xyz="-0.0080916 -0.00072376 0.036704"
+        rpy="0 0 0" />
+      <mass
+        value="0.2" />
+      <inertia
+        ixx="8.2755E-06"
+        ixy="1.0134E-07"
+        ixz="-4.3905E-08"
+        iyy="1.3404E-05"
+        iyz="4.4903E-08"
+        izz="1.4047E-05" />
+    </inertial>
+    <visual>
+      <origin
+        xyz="0 0 0"
+        rpy="0 0 0" />
+      <geometry>
+        <mesh
+          filename="package://urdf/kidsize_model/11th/meshes/neck_Link.STL" />
+      </geometry>
+      <material
+        name="">
+        <color
+          rgba="0.79216 0.81961 0.93333 1" />
+      </material>
+    </visual>
+    <collision>
+      <origin
+        xyz="0 0 0"
+        rpy="0 0 0" />
+      <geometry>
+        <mesh
+          filename="package://urdf/kidsize_model/11th/meshes/neck_Link.STL" />
       </geometry>
     </collision>
@@ -161,10 +161,10 @@
     type="revolute">
     <origin
-      xyz="0.021 0 0.1455"
+      xyz="0.021 0 0.1495"
       rpy="0 0 0" />
     <parent
       link="trunk_link" />
     <child
-      link="neck_link" />
+      link="neck_Link" />
     <axis
       xyz="0 0 1" />
@@ -182,15 +182,15 @@
     <inertial>
       <origin
-        xyz="0.00450345001830527 0.000595557219749025 0.0437931178446717"
-        rpy="0 0 0" />
-      <mass
-        value="0.0369714111760929" />
-      <inertia
-        ixx="4.12219607929375E-05"
-        ixy="-2.11945970555521E-07"
-        ixz="-3.31411440390918E-07"
-        iyy="2.13723182847917E-05"
-        iyz="1.1533174673443E-07"
-        izz="3.30603763976263E-05" />
+        xyz="0.00029663 -3.6886E-05 0.037704"
+        rpy="0 0 0" />
+      <mass
+        value="0.25" />
+      <inertia
+        ixx="3.0661E-05"
+        ixy="1.425E-10"
+        ixz="-4.6871E-08"
+        iyy="7.3036E-06"
+        iyz="1.441E-09"
+        izz="2.8273E-05" />
     </inertial>
     <visual>
@@ -205,5 +205,5 @@
         name="">
         <color
-          rgba="0.792156862745098 0.819607843137255 0.933333333333333 1" />
+          rgba="0.79216 0.81961 0.93333 1" />
       </material>
     </visual>
@@ -222,8 +222,8 @@
     type="revolute">
     <origin
-      xyz="0.00375 0 0.038997"
-      rpy="0 0 0" />
-    <parent
-      link="neck_link" />
+      xyz="0.00375 0 0.038"
+      rpy="0 0 0" />
+    <parent
+      link="neck_Link" />
     <child
       link="head_link" />
@@ -243,15 +243,15 @@
     <inertial>
       <origin
-        xyz="-4.38514420769698E-06 0.0304470101810646 -3.26963632026403E-06"
-        rpy="0 0 0" />
-      <mass
-        value="0.00527059117297288" />
-      <inertia
-        ixx="2.04107926809469E-06"
-        ixy="-2.4644073510579E-13"
-        ixz="5.52958211200573E-18"
-        iyy="1.81185180679179E-06"
-        iyz="6.83796280856436E-13"
-        izz="9.88237069335444E-07" />
+        xyz="0.0030363 0.036247 3.3909E-13"
+        rpy="0 0 0" />
+      <mass
+        value="0.004" />
+      <inertia
+        ixx="4.4633E-06"
+        ixy="-3.5249E-07"
+        ixz="1.2655E-20"
+        iyy="3.6085E-06"
+        iyz="4.0375E-20"
+        izz="2.7666E-06" />
     </inertial>
     <visual>
@@ -266,5 +266,5 @@
         name="">
         <color
-          rgba="0.792156862745098 0.819607843137255 0.933333333333333 1" />
+          rgba="0.79216 0.81961 0.93333 1" />
       </material>
     </visual>
@@ -283,5 +283,5 @@
     type="revolute">
     <origin
-      xyz="0 0.043997 0.14275"
+      xyz="0 0.0515 0.14675"
       rpy="0 0 0" />
     <parent
@@ -304,15 +304,15 @@
     <inertial>
       <origin
-        xyz="0.000824213036169134 3.05697836353036E-06 -0.0117057363764614"
-        rpy="0 0 0" />
-      <mass
-        value="0.0428406210150828" />
-      <inertia
-        ixx="1.05664351148523E-05"
-        ixy="-7.99382750150073E-12"
-        ixz="-1.04478903557772E-07"
-        iyy="1.1925604716193E-05"
-        iyz="1.91164074618392E-10"
-        izz="6.88581853258153E-06" />
+        xyz="-0.0021118 -2.0802E-07 -0.037458"
+        rpy="0 0 0" />
+      <mass
+        value="0.46" />
+      <inertia
+        ixx="7.4077E-05"
+        ixy="1.7432E-10"
+        ixz="-6.9326E-06"
+        iyy="8.1541E-05"
+        iyz="2.1903E-10"
+        izz="2.1686E-05" />
     </inertial>
     <visual>
@@ -325,7 +325,7 @@
       </geometry>
       <material
-        name="material">
-        <color
-          rgba="0.792156862745098 0.819607843137255 0.933333333333333 1" />
+        name="">
+        <color
+          rgba="0.79216 0.81961 0.93333 1" />
       </material>
     </visual>
@@ -344,5 +344,5 @@
     type="revolute">
     <origin
-      xyz="0 0.053997 -0.0010033"
+      xyz="0.02425 0.049 0"
       rpy="0 -1.5708 0" />
     <parent
@@ -351,4 +351,126 @@
       link="left_upper_arm_link" />
     <axis
+      xyz="-1 0 0" />
+    <limit
+      lower="${-pi*0.9}"
+      upper="${pi*0.9}"
+      effort="1000"
+      velocity="100" />
+    <dynamics
+      damping="0.0"
+      friction="0.7" />
+  </joint>
+  <link
+    name="left_middle_arm_link">
+    <inertial>
+      <origin
+        xyz="0.0007383 8.6844E-06 -0.047706"
+        rpy="0 0 0" />
+      <mass
+        value="0.24" />
+      <inertia
+        ixx="1.3032E-05"
+        ixy="-2.9073E-09"
+        ixz="1.3333E-07"
+        iyy="1.3674E-05"
+        iyz="-1.3074E-08"
+        izz="7.9361E-06" />
+    </inertial>
+    <visual>
+      <origin
+        xyz="0 0 0"
+        rpy="0 0 0" />
+      <geometry>
+        <mesh
+          filename="package://urdf/kidsize_model/11th/meshes/left_middle_arm_link.STL" />
+      </geometry>
+      <material
+        name="">
+        <color
+          rgba="0.79216 0.81961 0.93333 1" />
+      </material>
+    </visual>
+    <collision>
+      <origin
+        xyz="0 0 0"
+        rpy="0 0 0" />
+      <geometry>
+        <mesh
+          filename="package://urdf/kidsize_model/11th/meshes/left_middle_arm_link.STL" />
+      </geometry>
+    </collision>
+  </link>
+  <joint
+    name="left_middle_yaw"
+    type="revolute">
+    <origin
+      xyz="0.00575 0 -0.060331"
+      rpy="0 0 0" />
+    <parent
+      link="left_upper_arm_link" />
+    <child
+      link="left_middle_arm_link" />
+    <axis
+      xyz="0 0 -1" />
+    <limit
+      lower="${-pi*0.9}"
+      upper="${pi*0.9}"
+      effort="1000"
+      velocity="100" />
+    <dynamics
+      damping="0.0"
+      friction="0.7" />
+  </joint>
+  <link
+    name="left_lower_arm_link">
+    <inertial>
+      <origin
+        xyz="0.0076862 0.00892 -0.075914"
+        rpy="0 0 0" />
+      <mass
+        value="0.115" />
+      <inertia
+        ixx="3.4222E-05"
+        ixy="8.0645E-07"
+        ixz="5.5788E-06"
+        iyy="4.0879E-05"
+        iyz="1.6007E-06"
+        izz="1.2225E-05" />
+    </inertial>
+    <visual>
+      <origin
+        xyz="0 0 0"
+        rpy="0 0 0" />
+      <geometry>
+        <mesh
+          filename="package://urdf/kidsize_model/11th/meshes/left_lower_arm_link.STL" />
+      </geometry>
+      <material
+        name="">
+        <color
+          rgba="0.79216 0.81961 0.93333 1" />
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
File: urdf/kidsize_model/robocup_robot/robots/robocup.xacro (robot description, xacro)
@@ -17,20 +17,20 @@
 		</material>
   <!--link name="dummy">
-   </link-->
+    </link-->
   <link
     name="waist_link">
     <inertial>
       <origin
-        xyz="-0.010499 -4.8863E-05 0.35143"
-        rpy="0 0 0" />
-      <mass
-        value="0.16736" />
-      <inertia
-        ixx="0.00024686"
-        ixy="1.3146E-07"
-        ixz="-2.4647E-06"
-        iyy="8.0245E-05"
-        iyz="1.7402E-08"
-        izz="0.00028946" />
+        xyz="-0.00939428139224641 -4.60441121757915E-08 -0.000641732576416809"
+        rpy="0 0 0" />
+      <mass
+        value="0.210943942888859" />
+      <inertia
+        ixx="0.000341787200379464"
+        ixy="1.68848036086564E-10"
+        ixz="1.27321856491004E-06"
+        iyy="9.98074093608564E-05"
+        iyz="5.24058097864859E-12"
+        izz="0.000357999063478674" />
     </inertial>
     <visual>
@@ -45,5 +45,5 @@
         name="">
         <color
-          rgba="1 1 1 1" />
+          rgba="0.752941176470588 0.752941176470588 0.752941176470588 1" />
       </material>
     </visual>
@@ -69,15 +69,15 @@
     <inertial>
       <origin
-        xyz="0.01024 0.00011325 0.070848"
-        rpy="0 0 0" />
-      <mass
-        value="1" />
-      <inertia
-        ixx="0.0011025"
-        ixy="2.5029E-06"
-        ixz="6.7048E-05"
-        iyy="0.00089946"
-        iyz="2.1953E-07"
-        izz="0.00071841" />
+        xyz="-0.00207929488403977 -0.000148840580601717 0.09882913193458"
+        rpy="0 0 0" />
+      <mass
+        value="0.639632099418805" />
+      <inertia
+        ixx="0.00207382837512236"
+        ixy="7.20391665944275E-07"
+        ixz="-0.000145762768834737"
+        iyy="0.00159922346192907"
+        iyz="2.52085914196649E-06"
+        izz="0.00200543365155241" />
     </inertial>
     <visual>
@@ -92,920 +92,920 @@
         name="">
         <color
+          rgba="0.792156862745098 0.819607843137255 0.933333333333333 1" />
+      </material>
+    </visual>
+    <collision>
+      <origin
+        xyz="0 0 0"
+        rpy="0 0 0" />
+      <geometry>
+        <mesh
+          filename="package://urdf/kidsize_model/robocup_robot/meshes/trunk_link.STL" />
+      </geometry>
+    </collision>
+  </link>
+  <joint
+    name="waist_yaw_joint"
+    type="revolute">
+    <origin
+      xyz="0 0 0"
+      rpy="0 0 0" />
+    <parent
+      link="waist_link" />
+    <child
+      link="trunk_link" />
+    <axis
+      xyz="0 0 1" />
+    <limit
+      lower="${-pi}"
+      upper="${pi}"
+      effort="100"
+      velocity="5" />
+    <dynamics
+      friction="0.7"
+      damping="0.1" />
+  </joint>
+  <link
+    name="left_shoulder_link">
+    <inertial>
+      <origin
+        xyz="0.00303632774271406 0.0362469594639394 3.31679128606766E-15"
+        rpy="0 0 0" />
+      <mass
+        value="0.0085292893519016" />
+      <inertia
+        ixx="4.4633278691704E-06"
+        ixy="-3.52494995340182E-07"
+        ixz="-2.31421700758012E-20"
+        iyy="3.60847595287127E-06"
+        iyz="1.58823766686137E-21"
+        izz="2.76664423653777E-06" />
+    </inertial>
+    <visual>
+      <origin
+        xyz="0 0 0"
+        rpy="0 0 0" />
+      <geometry>
+        <mesh
+          filename="package://urdf/kidsize_model/robocup_robot/meshes/left_shoulder_link.STL" />
+      </geometry>
+      <material
+        name="">
+        <color
+          rgba="0.792156862745098 0.819607843137255 0.933333333333333 1" />
+      </material>
+    </visual>
+    <collision>
+      <origin
+        xyz="0 0 0"
+        rpy="0 0 0" />
+      <geometry>
+        <mesh
+          filename="package://urdf/kidsize_model/robocup_robot/meshes/left_shoulder_link.STL" />
+      </geometry>
+    </collision>
+  </link>
+  <joint
+    name="left_shoulder_pitch_joint"
+    type="revolute">
+    <origin
+      xyz="0 0.053 0.14675"
+      rpy="0 0 0" />
+    <parent
+      link="trunk_link" />
+    <child
+      link="left_shoulder_link" />
+    <axis
+      xyz="0 1 0" />
+    <limit
+      lower="${-pi}"
+      upper="${pi}"
+      effort="100"
+      velocity="5" />
+    <dynamics
+      friction="0.7"
+      damping="0.1" />
+  </joint>
+  <link
+    name="left_upper_arm_link">
+    <inertial>
+      <origin
+        xyz="0.000678411211440105 -1.8987570867858E-07 -0.0191217777296797"
+        rpy="0 0 0" />
+      <mass
+        value="0.0510794115590111" />
+      <inertia
+        ixx="3.13133402075074E-05"
+        ixy="-6.57973359323336E-12"
+        ixz="-3.53618283016186E-07"
+        iyy="3.06157554760576E-05"
+        iyz="2.63047056126239E-10"
+        izz="9.80852784205314E-06" />
+    </inertial>
+    <visual>
+      <origin
+        xyz="0 0 0"
+        rpy="0 0 0" />
+      <geometry>
+        <mesh
+          filename="package://urdf/kidsize_model/robocup_robot/meshes/left_upper_arm_link.STL" />
+      </geometry>
+      <material
+        name="">
+        <color
+          rgba="0.792156862745098 0.819607843137255 0.933333333333333 1" />
+      </material>
+    </visual>
+    <collision>
+      <origin
+        xyz="0 0 0"
+        rpy="0 0 0" />
+      <geometry>
+        <mesh
+          filename="package://urdf/kidsize_model/robocup_robot/meshes/left_upper_arm_link.STL" />
+      </geometry>
+    </collision>
+  </link>
+  <joint
+    name="left_upper_arm_roll_joint"
+    type="revolute">
+    <origin
+      xyz="0.02425 0.049 0"
+      rpy="0 -1.5708 0" />
+    <parent
+      link="left_shoulder_link" />
+    <child
+      link="left_upper_arm_link" />
+    <axis
+      xyz="-1 0 0" />
+    <limit
+      lower="${-pi}"
+      upper="${pi}"
+      effort="100"
+      velocity="5" />
+    <dynamics
+      friction="0.7"
+      damping="0.1" />
+  </joint>
+  <link
+    name="left_elbow_link">
+    <inertial>
+      <origin
+        xyz="1.85168757452225E-07 0.00233363841472187 -0.0273900365208956"
+        rpy="0 0 0" />
+      <mass
+        value="0.0523778400197291" />
+      <inertia
+        ixx="9.27211209059553E-05"
+        ixy="2.26333509945507E-11"
+        ixz="-3.43238744020251E-10"
+        iyy="9.36327197767988E-05"
+        iyz="6.86105678251835E-06"
+        izz="1.08163961495754E-05" />
+    </inertial>
+    <visual>
+      <origin
+        xyz="0 0 0"
+        rpy="0 0 0" />
+      <geometry>
+        <mesh
+          filename="package://urdf/kidsize_model/robocup_robot/meshes/left_elbow_link.STL" />
+      </geometry>
+      <material
+        name="">
+        <color
+          rgba="0.752941176470588 0.752941176470588 0.752941176470588 1" />
+      </material>
+    </visual>
+    <collision>
+      <origin
+        xyz="0 0 0"
+        rpy="0 0 0" />
+      <geometry>
+        <mesh
+          filename="package://urdf/kidsize_model/robocup_robot/meshes/left_elbow_link.STL" />
+      </geometry>
+    </collision>
+  </link>
+  <joint
+    name="left_elbow_pitch_joint"
+    type="revolute">
+    <origin
+      xyz="0 0 -0.10025"
+      rpy="0 0 0" />
+    <parent
+      link="left_upper_arm_link" />
+    <child
+      link="left_elbow_link" />
+    <axis
+      xyz="0 1 0" />
+    <limit
+      lower="${-pi}"
+      upper="${pi}"
+      effort="100"
+      velocity="5" />
+    <dynamics
+      friction="0.7"
+      damping="0.1" />
+  </joint>
+  <link
+    name="right_shoulder_link">
+    <inertial>
+      <origin
+        xyz="0.00303632774271398 -0.0362469594639394 9.57567358739198E-16"
+        rpy="0 0 0" />
+      <mass
+        value="0.0085292893519016" />
+      <inertia
+        ixx="4.4633278691704E-06"
+        ixy="3.5249499534018E-07"
+        ixz="-2.26133899466046E-23"
+        iyy="3.60847595287127E-06"
+        iyz="3.01602055369598E-21"
+        izz="2.76664423653777E-06" />
+    </inertial>
+    <visual>
+      <origin
+        xyz="0 0 0"
+        rpy="0 0 0" />
+      <geometry>
+        <mesh
+          filename="package://urdf/kidsize_model/robocup_robot/meshes/right_shoulder_link.STL" />
+      </geometry>
+      <material
+        name="">
+        <color
+          rgba="0.792156862745098 0.819607843137255 0.933333333333333 1" />
+      </material>
+    </visual>
+    <collision>
+      <origin
+        xyz="0 0 0"
+        rpy="0 0 0" />
+      <geometry>
+        <mesh
+          filename="package://urdf/kidsize_model/robocup_robot/meshes/right_shoulder_link.STL" />
+      </geometry>
+    </collision>
+  </link>
+  <joint
+    name="right_shoulder_pitch_joint"
+    type="revolute">
+    <origin
+      xyz="0 -0.053 0.14675"
+      rpy="0 0 0" />
+    <parent
+      link="trunk_link" />
+    <child
+      link="right_shoulder_link" />
+    <axis
+      xyz="0 -1 0" />
+    <limit
+      lower="${-pi}"
+      upper="${pi}"
+      effort="100"
+      velocity="5" />
+    <dynamics
+      friction="0.7"
+      damping="0.1" />
+  </joint>
+  <link
+    name="right_upper_arm_link">
+    <inertial>
+      <origin
+        xyz="0.000683044937076036 1.08215084787533E-05 -0.0193161303708199"
+        rpy="0 0 0" />
+      <mass
+        value="0.0511158524108051" />
+      <inertia
+        ixx="3.18475528264542E-05"
+        ixy="4.54446779241538E-10"
+        ixz="-4.48940731057538E-07"
+        iyy="3.11274405794203E-05"
+        iyz="3.94345652689599E-08"
+        izz="9.81721455090846E-06" />
+    </inertial>
+    <visual>
+      <origin
+        xyz="0 0 0"
+        rpy="0 0 0" />
+      <geometry>
+        <mesh
+          filename="package://urdf/kidsize_model/robocup_robot/meshes/right_upper_arm_link.STL" />
+      </geometry>
+      <material
+        name="">
+        <color
+          rgba="0.792156862745098 0.819607843137255 0.933333333333333 1" />
+      </material>
+    </visual>
+    <collision>
+      <origin
+        xyz="0 0 0"
+        rpy="0 0 0" />
+      <geometry>
+        <mesh
+          filename="package://urdf/kidsize_model/robocup_robot/meshes/right_upper_arm_link.STL" />
+      </geometry>
+    </collision>
+  </link>
+  <joint
+    name="right_upper_arm_roll_joint"
+    type="revolute">
+    <origin
+      xyz="0.02425 -0.049 0"
+      rpy="0 -1.5708 0" />
+    <parent
+      link="right_shoulder_link" />
+    <child
+      link="right_upper_arm_link" />
+    <axis
+      xyz="-1 0 0" />
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