Commit message: all project update models

File: urdf/kidsize_model/11th/robots/11th.xacro (robot description, xacro)
@@ -23,5 +23,5 @@
         rpy="0 0 0" />
       <mass
-        value="0.5" />
+        value="0.22475" />
       <inertia
         ixx="0.00037837"
@@ -63,5 +63,5 @@
         rpy="0 0 0" />
       <mass
-        value="1.3" />
+        value="0.26146" />
       <inertia
         ixx="0.0010729"
@@ -124,5 +124,5 @@
         rpy="0 0 0" />
       <mass
-        value="0.2" />
+        value="0.047879" />
       <inertia
         ixx="8.2755E-06"
@@ -185,5 +185,5 @@
         rpy="0 0 0" />
       <mass
-        value="0.25" />
+        value="0.049548" />
       <inertia
         ixx="3.0661E-05"
@@ -246,5 +246,5 @@
         rpy="0 0 0" />
       <mass
-        value="0.004" />
+        value="0.0085293" />
       <inertia
         ixx="4.4633E-06"
@@ -307,5 +307,5 @@
         rpy="0 0 0" />
       <mass
-        value="0.46" />
+        value="0.093248" />
       <inertia
         ixx="7.4077E-05"
@@ -368,5 +368,5 @@
         rpy="0 0 0" />
       <mass
-        value="0.24" />
+        value="0.047332" />
       <inertia
         ixx="1.3032E-05"
@@ -429,5 +429,5 @@
         rpy="0 0 0" />
       <mass
-        value="0.115" />
+        value="0.023059" />
       <inertia
         ixx="3.4222E-05"
@@ -490,5 +490,5 @@
         rpy="0 0 0" />
       <mass
-        value="0.04" />
+        value="0.0085293" />
       <inertia
         ixx="4.4633E-06"
@@ -551,5 +551,5 @@
         rpy="0 0 0" />
       <mass
-        value="0.46" />
+        value="0.093248" />
       <inertia
         ixx="7.4077E-05"
@@ -612,5 +612,5 @@
         rpy="0 0 0" />
       <mass
-        value="0.23" />
+        value="0.047295" />
       <inertia
         ixx="1.2988E-05"
@@ -673,5 +673,5 @@
         rpy="0 0 0" />
       <mass
-        value="0.115" />
+        value="0.023059" />
       <inertia
         ixx="3.4222E-05"
@@ -734,5 +734,5 @@
         rpy="0 0 0" />
       <mass
-        value="0.09" />
+        value="0.018738" />
       <inertia
         ixx="3.9876E-06"
@@ -795,5 +795,5 @@
         rpy="0 0 0" />
       <mass
-        value="0.46" />
+        value="0.093018" />
       <inertia
         ixx="2.4459E-05"
@@ -856,5 +856,5 @@
         rpy="0 0 0" />
       <mass
-        value="0.34" />
+        value="0.068207" />
       <inertia
         ixx="5.7966E-05"
@@ -917,5 +917,5 @@
         rpy="0 0 0" />
       <mass
-        value="0.007" />
+        value="0.015114" />
       <inertia
         ixx="2.1026E-05"
@@ -978,5 +978,5 @@
         rpy="0 0 0" />
       <mass
-        value="0.46" />
+        value="0.093018" />
       <inertia
         ixx="2.4459E-05"
@@ -1039,5 +1039,5 @@
         rpy="0 0 0" />
       <mass
-        value="0.16" />
+        value="0.032328" />
       <inertia
         ixx="1.2045E-05"
@@ -1100,5 +1100,5 @@
         rpy="0 0 0" />
       <mass
-        value="0.09" />
+        value="0.018738" />
       <inertia
         ixx="3.9876E-06"
@@ -1161,5 +1161,5 @@
         rpy="0 0 0" />
       <mass
-        value="0.46" />
+        value="0.093018" />
       <inertia
         ixx="2.4459E-05"
@@ -1222,5 +1222,5 @@
         rpy="0 0 0" />
       <mass
-        value="0.34" />
+        value="0.068207" />
       <inertia
         ixx="5.7966E-05"
@@ -1283,5 +1283,5 @@
         rpy="0 0 0" />
       <mass
-        value="0.07" />
+        value="0.015114" />
       <inertia
         ixx="2.1026E-05"
@@ -1344,5 +1344,5 @@
         rpy="0 0 0" />
       <mass
-        value="0.46" />
+        value="0.093018" />
       <inertia
         ixx="2.4459E-05"
@@ -1405,5 +1405,5 @@
         rpy="0 0 0" />
       <mass
-        value="0.16" />
+        value="0.032328" />
       <inertia
         ixx="1.2045E-05"
@@ -1799,5 +1799,5 @@
   </gazebo> -->
 <gazebo reference="camera_link">
-<material>Gazebo/Black</material>
+  <material>Gazebo/DarkGrey</material>
     <sensor type="camera" name="camera1">
       <visualize>0</visualize>
@@ -1841,27 +1841,32 @@
 </gazebo>
 		<!-- Gazebo links -->
+    <gazebo reference="head_link">
+			<material>Gazebo/DarkGrey</material>
+		</gazebo>
 		<gazebo reference="trunk_link">
-			<material>Gazebo/White</material>
-		</gazebo>
-                <gazebo reference="waist_link">
-			<material>Gazebo/White</material>
+			<material>Gazebo/DarkGrey</material>
+		</gazebo>
+    <gazebo reference="waist_link">
+			<material>Gazebo/DarkGrey</material>
 		</gazebo>
 		<gazebo reference="left_hip_yaw_link">
-			<material>Gazebo/White</material>
+			<material>Gazebo/DarkGrey</material>
 		</gazebo>
 		<gazebo reference="left_hip_roll_link">
-			<material>Gazebo/Black</material>
+			<material>Gazebo/FlatBlack</material>
 		</gazebo>
 		<gazebo reference="left_thigh_link">
-			<material>Gazebo/White</material>
+			<material>Gazebo/DarkGrey</material>
 		</gazebo>
 		<gazebo reference="left_shank_link">
-			<material>Gazebo/White</material>
+			<material>Gazebo/DarkGrey</material>
 		</gazebo>
 		<gazebo reference="left_ankle_link">
-			<material>Gazebo/Black</material>
+			<material>Gazebo/FlatBlack</material>
+      <mu1>100000.0</mu1>
+			<mu2>100000.0</mu2>
 		</gazebo>
 		<gazebo reference="left_foot_link">
-			<material>Gazebo/FlatBlack</material>
+			<material>Gazebo/DarkGrey</material>
 			<kp>1000000.0</kp>
 			<kd>100.0</kd>
@@ -1873,32 +1878,40 @@
 		</gazebo>
 		<gazebo reference="left_shoulder_pitch_link">
-			<material>Gazebo/White</material>
+			<material>Gazebo/DarkGrey</material>
 		</gazebo>
 		<gazebo reference="left_upper_arm_link">
-			<material>Gazebo/White</material>
-		</gazebo>
-                <gazebo reference="left_middle_arm_link">
-			<material>Gazebo/White</material>
+			<material>Gazebo/DarkGrey</material>
+      <mu1>100000.0</mu1>
+			<mu2>100000.0</mu2>
+		</gazebo>
+    <gazebo reference="left_middle_arm_link">
+			<material>Gazebo/FlatBlack</material>
+      <mu1>100000.0</mu1>
+			<mu2>100000.0</mu2>
 		</gazebo>
 		<gazebo reference="left_lower_arm_link">
-			<material>Gazebo/White</material>
+			<material>Gazebo/DarkGrey</material>
+      <mu1>100000.0</mu1>
+			<mu2>100000.0</mu2>
 		</gazebo>
 		<gazebo reference="right_hip_yaw_link">
-			<material>Gazebo/White</material>
+			<material>Gazebo/DarkGrey</material>
 		</gazebo>
 		<gazebo reference="right_hip_roll_link">
-			<material>Gazebo/Black</material>
+			<material>Gazebo/FlatBlack</material>
 		</gazebo>
 		<gazebo reference="right_thigh_link">
-			<material>Gazebo/White</material>
+			<material>Gazebo/DarkGrey</material>
 		</gazebo>
 		<gazebo reference="right_shank_link">
-			<material>Gazebo/White</material>
+			<material>Gazebo/DarkGrey</material>
 		</gazebo>
 		<gazebo reference="right_ankle_link">
-			<material>Gazebo/Black</material>
+			<material>Gazebo/FlatBlack</material>
+      <mu1>100000.0</mu1>
+			<mu2>100000.0</mu2>
 		</gazebo>
 		<gazebo reference="right_foot_link">
-			<material>Gazebo/FlatBlack</material>
+			<material>Gazebo/DarkGrey</material>
 			<kp>1000000.0</kp>
 			<kd>100.0</kd>
@@ -1910,17 +1923,23 @@
 		</gazebo>
 		<gazebo reference="right_shoulder_pitch_link">
-			<material>Gazebo/White</material>
+			<material>Gazebo/DarkGrey</material>
 		</gazebo>
 		<gazebo reference="right_upper_arm_link">
-			<material>Gazebo/White</material>
-		</gazebo>
-                <gazebo reference="right_middle_arm_link">
-			<material>Gazebo/White</material>
+      <material>Gazebo/DarkGrey</material>
+      <mu1>100000.0</mu1>
+			<mu2>100000.0</mu2>
+		</gazebo>
+    <gazebo reference="right_middle_arm_link">
+			<material>Gazebo/FlatBlack</material>
+      <mu1>100000.0</mu1>
+			<mu2>100000.0</mu2>
 		</gazebo>
 		<gazebo reference="right_lower_arm_link">
-			<material>Gazebo/White</material>
-		</gazebo>
-		<gazebo reference="neck_link">
-			<material>Gazebo/Black</material>
+			<material>Gazebo/DarkGrey</material>
+      <mu1>100000.0</mu1>
+			<mu2>100000.0</mu2>
+		</gazebo>
+		<gazebo reference="neck_Link">
+			<material>Gazebo/FlatBlack</material>
 		</gazebo>
     <gazebo reference="trunk_link">
