Commit message: add balance control & IMU

File: urdf/kidsize_model/robocup_robot/robots/robocup1111.xacro (robot description, xacro)
@@ -17,20 +17,20 @@
 		</material>
   <!--link name="dummy">
-    </link-->
+   </link-->
   <link
     name="waist_link">
     <inertial>
       <origin
-        xyz="-0.00939428139224641 -4.60441121757915E-08 -0.000641732576416809"
-        rpy="0 0 0" />
-      <mass
-        value="0.210943942888859" />
-      <inertia
-        ixx="0.000341787200379464"
-        ixy="1.68848036086564E-10"
-        ixz="1.27321856491004E-06"
-        iyy="9.98074093608564E-05"
-        iyz="5.24058097864859E-12"
-        izz="0.000357999063478674" />
+        xyz="-0.010499 -4.8863E-05 0.35143"
+        rpy="0 0 0" />
+      <mass
+        value="0.16736" />
+      <inertia
+        ixx="0.00024686"
+        ixy="1.3146E-07"
+        ixz="-2.4647E-06"
+        iyy="8.0245E-05"
+        iyz="1.7402E-08"
+        izz="0.00028946" />
     </inertial>
     <visual>
@@ -45,5 +45,5 @@
         name="">
         <color
-          rgba="0.752941176470588 0.752941176470588 0.752941176470588 1" />
+          rgba="1 1 1 1" />
       </material>
     </visual>
@@ -69,15 +69,15 @@
     <inertial>
       <origin
-        xyz="-0.00207929488403977 -0.000148840580601717 0.09882913193458"
-        rpy="0 0 0" />
-      <mass
-        value="0.639632099418805" />
-      <inertia
-        ixx="0.00207382837512236"
-        ixy="7.20391665944275E-07"
-        ixz="-0.000145762768834737"
-        iyy="0.00159922346192907"
-        iyz="2.52085914196649E-06"
-        izz="0.00200543365155241" />
+        xyz="0.01024 0.00011325 0.070848"
+        rpy="0 0 0" />
+      <mass
+        value="1" />
+      <inertia
+        ixx="0.0011025"
+        ixy="2.5029E-06"
+        ixz="6.7048E-05"
+        iyy="0.00089946"
+        iyz="2.1953E-07"
+        izz="0.00071841" />
     </inertial>
     <visual>
@@ -92,920 +92,920 @@
         name="">
         <color
+          rgba="1 1 1 1" />
+      </material>
+    </visual>
+    <collision>
+      <origin
+        xyz="0 0 0"
+        rpy="0 0 0" />
+      <geometry>
+        <mesh
+          filename="package://urdf/kidsize_model/robocup_robot/meshes/trunk_link.STL" />
+      </geometry>
+    </collision>
+  </link>
+  <joint
+    name="waist_yaw_joint"
+    type="revolute">
+    <origin
+      xyz="-0.00045 0 0.3865"
+      rpy="0 0 0" />
+    <parent
+      link="waist_link" />
+    <child
+      link="trunk_link" />
+    <axis
+      xyz="0 0 1" />
+    <limit
+      lower="${-pi}"
+      upper="${pi}"
+      effort="100"
+      velocity="5" />
+    <dynamics
+      friction="0.7"
+      damping="0.1" />
+  </joint>
+  <link
+    name="left_shoulder_link">
+    <inertial>
+      <origin
+        xyz="-3.72604127105386E-06 0.0297911074033573 -0.00461915163355214"
+        rpy="0 0 0" />
+      <mass
+        value="0.00596009981158904" />
+      <inertia
+        ixx="1.26246219599389E-06"
+        ixy="-1.72427552349869E-11"
+        ixz="6.85742889803387E-12"
+        iyy="2.28404971724678E-06"
+        iyz="3.17827997088839E-07"
+        izz="2.37194480329819E-06" />
+    </inertial>
+    <visual>
+      <origin
+        xyz="0 0 0"
+        rpy="0 0 0" />
+      <geometry>
+        <mesh
+          filename="package://urdf/kidsize_model/robocup_robot/meshes/left_shoulder_link.STL" />
+      </geometry>
+      <material
+        name="">
+        <color
+          rgba="1 1 1 1" />
+      </material>
+    </visual>
+    <collision>
+      <origin
+        xyz="0 0 0"
+        rpy="0 0 0" />
+      <geometry>
+        <mesh
+          filename="package://urdf/kidsize_model/robocup_robot/meshes/left_shoulder_link.STL" />
+      </geometry>
+    </collision>
+  </link>
+  <joint
+    name="left_shoulder_pitch_joint"
+    type="revolute">
+    <origin
+      xyz="0 0.043997 0.10474"
+      rpy="0 0 0" />
+    <parent
+      link="trunk_link" />
+    <child
+      link="left_shoulder_link" />
+    <axis
+      xyz="0 1 0" />
+    <limit
+      lower="${-pi}"
+      upper="${pi}"
+      effort="100"
+      velocity="5" />
+    <dynamics
+      friction="0.7"
+      damping="0.1" />
+  </joint>
+  <link
+    name="left_upper_arm_link">
+    <inertial>
+      <origin
+        xyz="0.000678411211435796 0.000489810124291307 -0.0191217777296809"
+        rpy="0 0 0" />
+      <mass
+        value="0.0510794115590112" />
+      <inertia
+        ixx="3.1313340207507E-05"
+        ixy="-6.57973357844028E-12"
+        ixz="-3.53618283019284E-07"
+        iyy="3.06157554760573E-05"
+        iyz="2.63047056443396E-10"
+        izz="9.80852784205324E-06" />
+    </inertial>
+    <visual>
+      <origin
+        xyz="0 0 0"
+        rpy="0 0 0" />
+      <geometry>
+        <mesh
+          filename="package://urdf/kidsize_model/robocup_robot/meshes/left_upper_arm_link.STL" />
+      </geometry>
+      <material
+        name="">
+        <color
+          rgba="1 1 1 1" />
+      </material>
+    </visual>
+    <collision>
+      <origin
+        xyz="0 0 0"
+        rpy="0 0 0" />
+      <geometry>
+        <mesh
+          filename="package://urdf/kidsize_model/robocup_robot/meshes/left_upper_arm_link.STL" />
+      </geometry>
+    </collision>
+  </link>
+  <joint
+    name="left_upper_arm_roll_joint"
+    type="revolute">
+    <origin
+      xyz="0 0.04851 -0.011774"
+      rpy="0 0 0" />
+    <parent
+      link="left_shoulder_link" />
+    <child
+      link="left_upper_arm_link" />
+    <axis
+      xyz="1 0 0" />
+    <limit
+      lower="${-pi}"
+      upper="${pi}"
+      effort="100"
+      velocity="5" />
+    <dynamics
+      friction="0.7"
+      damping="0.1" />
+  </joint>
+  <link
+    name="left_elbow_link">
+    <inertial>
+      <origin
+        xyz="-0.000489816928373502 0.0024374519516502 -0.0293208681909612"
+        rpy="0 0 0" />
+      <mass
+        value="0.0529778400197291" />
+      <inertia
+        ixx="0.000109530121626401"
+        ixy="2.36402125251114E-11"
+        ixz="-3.61965391083585E-10"
+        iyy="0.000110422928141888"
+        iyz="7.78807652504947E-06"
+        izz="1.08976885049728E-05" />
+    </inertial>
+    <visual>
+      <origin
+        xyz="0 0 0"
+        rpy="0 0 0" />
+      <geometry>
+        <mesh
+          filename="package://urdf/kidsize_model/robocup_robot/meshes/left_botton_arm_link.STL" />
+      </geometry>
+      <material
+        name="">
+        <color
+          rgba="1 1 1 1" />
+      </material>
+    </visual>
+    <collision>
+      <origin
+        xyz="0 0 0"
+        rpy="0 0 0" />
+      <geometry>
+        <mesh
+          filename="package://urdf/kidsize_model/robocup_robot/meshes/left_botton_arm_link.STL" />
+      </geometry>
+    </collision>
+  </link>
+  <joint
+    name="left_elbow_pitch_joint"
+    type="revolute">
+    <origin
+      xyz="0.00049 0.00049 -0.10025"
+      rpy="0 0 0" />
+    <parent
+      link="left_upper_arm_link" />
+    <child
+      link="left_elbow_link" />
+    <axis
+      xyz="0 1 0" />
+    <limit
+      lower="${-pi}"
+      upper="${pi}"
+      effort="100"
+      velocity="5" />
+    <dynamics
+      friction="0.7"
+      damping="0.1" />
+  </joint>
+  <link
+    name="right_shoulder_link">
+    <inertial>
+      <origin
+        xyz="3.7260412035388E-06 -0.0297911074033573 -0.00363915163355155"
+        rpy="0 0 0" />
+      <mass
+        value="0.005960099811589" />
+      <inertia
+        ixx="1.26246219599387E-06"
+        ixy="-1.72427551985748E-11"
+        ixz="-6.85742905110232E-12"
+        iyy="2.28404971724675E-06"
+        iyz="-3.17827997088837E-07"
+        izz="2.37194480329818E-06" />
+    </inertial>
+    <visual>
+      <origin
+        xyz="0 0 0"
+        rpy="0 0 0" />
+      <geometry>
+        <mesh
+          filename="package://urdf/kidsize_model/robocup_robot/meshes/right_shoulder_link.STL" />
+      </geometry>
+      <material
+        name="">
+        <color
+          rgba="1 1 1 1" />
+      </material>
+    </visual>
+    <collision>
+      <origin
+        xyz="0 0 0"
+        rpy="0 0 0" />
+      <geometry>
+        <mesh
+          filename="package://urdf/kidsize_model/robocup_robot/meshes/right_shoulder_link.STL" />
+      </geometry>
+    </collision>
+  </link>
+  <joint
+    name="right_shoulder_pitch_joint"
+    type="revolute">
+    <origin
+      xyz="0 -0.044003 0.10376"
+      rpy="0 0 0" />
+    <parent
+      link="trunk_link" />
+    <child
+      link="right_shoulder_link" />
+    <axis
+      xyz="0 -1 0" />
+    <limit
+      lower="${-pi}"
+      upper="${pi}"
+      effort="100"
+      velocity="5" />
+    <dynamics
+      friction="0.7"
+      damping="0.1" />
+  </joint>
+  <link
+    name="right_upper_arm_link">
+    <inertial>
+      <origin
+        xyz="0.000678411211443852 -0.000490189875708882 -0.0191217777296777"
+        rpy="0 0 0" />
+      <mass
+        value="0.0510794115590111" />
+      <inertia
+        ixx="3.13133402075077E-05"
+        ixy="-6.57973359766917E-12"
+        ixz="-3.53618283010164E-07"
+        iyy="3.06157554760577E-05"
+        iyz="2.63047055845698E-10"
+        izz="9.80852784205294E-06" />
+    </inertial>
+    <visual>
+      <origin
+        xyz="0 0 0"
+        rpy="0 0 0" />
+      <geometry>
+        <mesh
+          filename="package://urdf/kidsize_model/robocup_robot/meshes/right_upper_arm_link.STL" />
+      </geometry>
+      <material
+        name="">
+        <color
+          rgba="1 1 1 1" />
+      </material>
+    </visual>
+    <collision>
+      <origin
+        xyz="0 0 0"
+        rpy="0 0 0" />
+      <geometry>
+        <mesh
+          filename="package://urdf/kidsize_model/robocup_robot/meshes/right_upper_arm_link.STL" />
+      </geometry>
+    </collision>
+  </link>
+  <joint
+    name="right_upper_arm_roll_joint"
+    type="revolute">
+    <origin
+      xyz="0 -0.04851 -0.010794"
+      rpy="0 0 0" />
+    <parent
+      link="right_shoulder_link" />
+    <child
+      link="right_upper_arm_link" />
+    <axis
+      xyz="1 0 0" />
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